Commit message: fixed arm position on the robot back in the urdf

File: source/GO2_policy/GO2_policy/robots/description_files/go2_with_d1_550_description/go2_with_d1_550_description.urdf (robot description, URDF)
Before this commit: robot go2_with_d1_550_description, 51 links, 50 joints
Links:
- added link arm_mount_plate, mass 0.5; collision box size=0.20 0.10 0.015; visual box size=0.20 0.10 0.015
Joints:
- added joint arm_plate_joint: type fixed, parent base, child arm_mount_plate, origin xyz=0 0 0.065 rpy=0 0 0
- joint arm_mount_joint: origin xyz=0.1 0 0.05 rpy=0 0 0 -> xyz=0 0 0.0075 rpy=0 0 0; parent base -> arm_mount_plate
